File: _autosave-Numpad.kicad_pcb (KiCad board)
At the start: 2 copper layers, 54 parts, among them J1 USB_B_Mini, SW0 MXSwitch, SW1 MXSwitch, SW2 MXSwitch, SW3 MXSwitch, SW4 MXSwitch, SW5 MXSwitch, SW6 MXSwitch, SW7 MXSwitch, SW8 MXSwitch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

Commit message: ignore bak files, went bak to standard pcb orientation
Parts:
- added R5: 330, Resistor_SMD:R_1206_3216Metric_Pad1.42x1.75mm_HandSolder, F.Cu at (50.8, 58.4)
- D0, D1, D2, D3, D4, D5, D6, D7, D8, D9, DAst1, DDel1, DDiv1, DEnt1, DNum1, DPls1: value D_Small -> 1N4148W
- R4: value 10K -> 1K
- SW0: value MXSwitch -> 0
- SW1: value MXSwitch -> 1
- SW2: value MXSwitch -> 2
- SW3: value MXSwitch -> 3
- SW4: value MXSwitch -> 4
- SW5: value MXSwitch -> 5
- SW6: value MXSwitch -> 6
- SW7: value MXSwitch -> 7
- SW8: value MXSwitch -> 8
- SW9: value MXSwitch -> 9
- SWAst1: value MXSwitch -> Ast
- SWDel1: value MXSwitch -> Del
- SWDiv1: value MXSwitch -> Div
- SWEnt1: value MXSwitch -> Ent
- SWMns1: value MXSwitch -> Mns
- SWNum1: value MXSwitch -> Num
- SWPls1: value MXSwitch -> Pls
- moved C7 191.4 mm to (16.5, 45.7)
- moved SWRst1 191.4 mm to (20.3, 118.1)
- moved C2 191.4 mm to (17.8, 85.1)
- moved C3 191.4 mm to (17.8, 95.2)
- moved C5 191.4 mm to (21.6, 45.7)
- moved C6 191.4 mm to (19.1, 45.7)
- moved C8 191.4 mm to (14.0, 45.7)
- moved D3 191.4 mm to (15.2, 102.9)
- moved J1 191.4 mm to (17.8, 36.8)
- moved R3 191.4 mm to (22.9, 52.1)
- moved R4 191.4 mm to (13.3, 52.1)
- moved Y1 191.4 mm to (17.8, 90.2)
- moved DNum1 151.8 mm to (92.7, 52.7)
- moved DDiv1 149.9 mm to (75.6, 50.2)
- moved D0 143.6 mm to (91.4, 125.7)
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Connections:
- C1 pad 2: GND -> Net-(C1-Pad2)
- SWRst1 pad 2: GND -> Net-(C1-Pad2)
